Commit message: fix: Fix joint position

File: mycobot_description/urdf/mycobot.urdf (robot description, URDF)
Before this commit: robot mycobot, 8 links, 7 joints
Joints:
- joint joint5: origin xyz=0.0288 0 0.02976 rpy=0 0 0 -> xyz=0.0298 0 0.02876 rpy=0 0 0

Commit message: refactor: Reformat

File: mycobot_description/urdf/mycobot.urdf (robot description, URDF)
Before this commit: robot mycobot, 8 links, 7 joints
Joints:
- joint base_joint: origin (none) -> xyz=0 0 0 rpy=0 0 1.57

Commit message: fix: Fix URDF model (#1)
* fix: Fix joint position

* fix: Fix link size

* refactor: Reformat URDF

File: mycobot_description/urdf/mycobot.urdf (robot description, URDF)
Before this commit: robot mycobot, 8 links, 7 joints
Joints:
- joint base_joint: origin (none) -> xyz=0 0 0 rpy=0 0 1.57
- joint joint5: origin xyz=0.0288 0 0.02976 rpy=0 0 0 -> xyz=0.0298 0 0.02876 rpy=0 0 0

Commit message: feat: Use realistic texture
Import dae files from elephantrobotics/mycobot_ros

File: mycobot_description/urdf/mycobot.urdf (robot description, URDF)
Before this commit: robot mycobot, 8 links, 7 joints
Links:
- link link6_flange: geometry visual mesh filename=package://mycobot_description/meshes/dae/link7.dae
Joints:
- joint base_joint: origin xyz=0 0 0 rpy=0 0 1.57 -> xyz=0 0 0 rpy=0 0 3.14
- joint joint1: limit lower=-3.14 upper=3.14159 effort=1000.0 velocity=0 -> lower=-2.88 upper=2.88 effort=1000.0 velocity=0; origin xyz=0 0 0.0706 rpy=0 0 0 -> xyz=0 0 0.13156 rpy=0 0 0
- joint joint2: axis 1 0 0 -> 0 0 1; limit lower=-3.14 upper=3.14159 effort=1000.0 velocity=0 -> lower=-2.88 upper=2.88 effort=1000.0 velocity=0; origin xyz=0.03256 0 0.05976 rpy=0 0 0 -> xyz=0 0 -0.001 rpy=0 1.57 -1.57
- joint joint3: axis 1 0 0 -> 0 0 1; limit lower=-3.14 upper=3.14159 effort=1000.0 velocity=0 -> lower=-2.88 upper=2.88 effort=1000.0 velocity=0; origin xyz= 0.00272 0 0.1104 rpy=0 0 0 -> xyz=-0.1104 0 0 rpy=0 0 0
- joint joint4: axis 1 0 0 -> 0 0 1; limit lower=-3.14 upper=3.14159 effort=1000.0 velocity=0 -> lower=-2.88 upper=2.88 effort=1000.0 velocity=0; origin xyz=-0.00164 0 0.096 rpy=0 0 0 -> xyz=-0.0965 0 0.0641 rpy=0 0 -1.57
- joint joint5: limit lower=-3.14 upper=3.14159 effort=1000.0 velocity=0 -> lower=-2.88 upper=2.88 effort=1000.0 velocity=0; origin xyz=0.0298 0 0.02876 rpy=0 0 0 -> xyz=0 -0.07318 0 rpy=1.5708 -1.5708 0
- joint joint6: axis 0 1 0 -> 0 0 1; limit lower=-3.14 upper=3.14159 effort=1000.0 velocity=0 -> lower=-3.05 upper=3.05 effort=1000.0 velocity=0; origin xyz=0 0.0456 0.03792 rpy=0 0 0 -> xyz=0 0.0456 0 rpy=-1.57 0 0

File: mycobot_description/urdf/mycobot.xacro (robot description, xacro)
@@ -26,5 +26,6 @@
       <visual>
         <geometry>
-          <mesh filename="package://mycobot_description/meshes/stl/visual/link1.stl" />
+          <mesh filename="package://mycobot_description/meshes/dae/link1.dae" />
+          <!-- <mesh filename="package://mycobot_description/meshes/stl/visual/link1.stl" /> -->
         </geometry>
         <origin xyz="0 0 0" rpy="0 0 0" />
@@ -47,5 +48,6 @@
       <visual>
         <geometry>
-          <mesh filename="package://mycobot_description/meshes/stl/visual/link2.stl" />
+          <mesh filename="package://mycobot_description/meshes/dae/link2.dae" />
+          <!-- <mesh filename="package://mycobot_description/meshes/stl/visual/link2.stl" /> -->
         </geometry>
         <origin xyz="0 0 0" rpy="0 0 0" />
@@ -68,5 +70,6 @@
       <visual>
         <geometry>
-          <mesh filename="package://mycobot_description/meshes/stl/visual/link3.stl" />
+          <mesh filename="package://mycobot_description/meshes/dae/link3.dae" />
+          <!-- <mesh filename="package://mycobot_description/meshes/stl/visual/link3.stl" /> -->
         </geometry>
         <origin xyz="0 0 0" rpy="0 0 0" />
@@ -89,5 +92,6 @@
       <visual>
         <geometry>
-          <mesh filename="package://mycobot_description/meshes/stl/visual/link4.stl" />
+          <mesh filename="package://mycobot_description/meshes/dae/link4.dae" />
+          <!-- <mesh filename="package://mycobot_description/meshes/stl/visual/link4.stl" /> -->
         </geometry>
         <origin xyz="0 0 0" rpy="0 0 0" />
@@ -110,5 +114,6 @@
       <visual>
         <geometry>
-          <mesh filename="package://mycobot_description/meshes/stl/visual/link5.stl" />
+          <mesh filename="package://mycobot_description/meshes/dae/link5.dae" />
+          <!-- <mesh filename="package://mycobot_description/meshes/stl/visual/link5.stl" /> -->
         </geometry>
         <origin xyz="0 0 0" rpy="0 0 0" />
@@ -120,5 +125,5 @@
           <!-- <mesh filename="package://mycobot_description/meshes/stl/visual/link5.stl" /> -->
         </geometry>
-        <origin xyz="0 0 0" rpy="0 0 0" />
+        <origin xyz="0.004 0 0" rpy="0 0 0" />
       </collision>
       <inertial>
@@ -131,5 +136,6 @@
       <visual>
         <geometry>
-          <mesh filename="package://mycobot_description/meshes/stl/visual/link6.stl" />
+          <mesh filename="package://mycobot_description/meshes/dae/link6.dae" />
+          <!-- <mesh filename="package://mycobot_description/meshes/stl/visual/link6.stl" /> -->
         </geometry>
         <origin xyz="0 0 0 " rpy="0 0 0" />
@@ -152,5 +158,6 @@
       <visual>
         <geometry>
-          <cylinder length="0.005" radius="0.02" />
+          <!-- <cylinder length="0.005" radius="0.02" /> -->
+          <mesh filename="package://mycobot_description/meshes/dae/link7.dae" />
         </geometry>
         <origin xyz="0 0.0025 0" rpy="${M_PI/2} 0 0" />
@@ -159,10 +166,10 @@
       <collision>
         <geometry>
-          <cylinder length="0.005" radius="0.02" />
-        </geometry>
-        <origin xyz="0 0.0025 0" rpy="${M_PI/2} 0 0" />
-      </collision>
-      <inertial>
-        <origin xyz="0 0.0025 0" rpy="${M_PI/2} 0 0" />
+          <cylinder length="0.013" radius="0.02" />
+        </geometry>
+        <origin xyz="0 -0.004 0" rpy="${M_PI/2} 0 0" />
+      </collision>
+      <inertial>
+        <origin xyz="0 -0.004 0" rpy="${M_PI/2} 0 0" />
         <mass value="0.1" />
         <xacro:cylinder_inertia m="0.1" r="0.02" h="0.005" />
@@ -190,5 +197,5 @@
       <parent link="${mycobot_link_3}" />
       <child link="${mycobot_link_4}" />
-      <origin xyz=" 0.00272 0 0.1104" rpy="0 0 0" />
+      <origin xyz="0 0 0.1104" rpy="0 0 0" />
       <dynamics damping="1.0e-6" friction="2.0e-1" />
     </joint>
@@ -206,5 +213,5 @@
       <parent link="${mycobot_link_5}" />
       <child link="${mycobot_link_6}" />
-      <origin xyz="0.0298 0 0.02876" rpy="0 0 0" />
+      <origin xyz="0.034 0 0.035" rpy="0 0 0" />
       <dynamics damping="1.0e-6" friction="2.0e-1" />
     </joint>
